File: Arduino Minimal Design.kicad_sch (KiCad schematic)
At the start: 33 parts, among them J1 Conn_01x09_Pin, J2 Conn_01x09_Pin, J3 Conn_01x09_Pin, J4 USB_OTG, SW1 SW_Omron_B3FS, U1 LM1117DT-3.3, U2 ATmega328P-M, U3 CH340E, Y1 16 MHz

Commit message: Adding Images
Other:
- company: (none) -> Home Electronics
- title: (none) -> Arduino Minimal Design
Changed lines of the file:
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@@
 	(generator_version "9.0")
 	(paper "A4")
+	(title_block
+		(title "Arduino Minimal Design")
+		(date "2026-03-13")
+		(company "Home Electronics")
+	)
 	(rectangle
 		(start 13.208 14.732)
